File: Jam Week/Friendship Pendant.sch (EAGLE design)
At the start: 2 parts, among them IC1 LM556D, IC2 LM556D

Commit message: Worked on eagle more
Parts:
- added C1, C2, C3, C4, C5: .01uF, rcl:C-USC0805
- added C6, C7: 100uF, rcl:C-USC0805
- added R1: 28.7K, rcl:R-US_R0805
- added R10, R17, R18, R19, R4: 10K, rcl:R-US_R0805
- added R11, R12: 30, rcl:R-US_R0805
- added R14: 15, rcl:R-US_R0805
- added R16, R9: 1K, rcl:R-US_R0805
- added R2: 1.1K, rcl:R-US_R0805
- added R3: 3.65K, rcl:R-US_R0805
- added R5: 1.87K, rcl:R-US_R0805
- added R6: 619K, rcl:R-US_R0805
- added R7: 1.24K, rcl:R-US_R0805
- added R8: 562, rcl:R-US_R0805
Connections:
- new net N$1: R2.1, R3.2
- new net N$2: R6.1, R7.2
